File: pcb/BrewPilot.kicad_sch (KiCad schematic)
At the start: 19 parts, among them K1 G3MB-202P DC5, K2 G3MB-202P DC5, K3 G3MB-202P DC5, K4 G3MB-202P DC5, K5 G3MB-202P DC5, K6 G3MB-202P DC5, Q1 BC547, Q2 BC547, Q3 BC547, Q4 BC547, Q5 BC547, Q6 BC547, U1 esp32

Commit message: added more stuff
Parts:
- removed K6: G3MB-202P DC5, G3MB-202P DC5_OMR, symbol new_local:G3MB-202P_DC5
- removed Q6: BC547, Package_TO_SOT_THT:TO-92_Inline, symbol Transistor_BJT:BC547
- removed R5: R, Resistor_THT:R_Axial_DIN0207_L6.3mm_D2.5mm_P7.62mm_Horizontal, symbol Device:R
- added J1: 5V Power, TerminalBlock_Phoenix:TerminalBlock_Phoenix_MKDS-1-2-3.81_1x02_P3.81mm_Horizontal, symbol Connector:Screw_Terminal_01x02
- added J2: Flow Meter Group One, TerminalBlock_Phoenix:TerminalBlock_Phoenix_MKDS-1-3-3.81_1x03_P3.81mm_Horizontal, symbol Connector:Screw_Terminal_01x03
- added J3: Flow Meter Group Two, TerminalBlock_Phoenix:TerminalBlock_Phoenix_MKDS-1-3-3.81_1x03_P3.81mm_Horizontal, symbol Connector:Screw_Terminal_01x03
- added J4: FlexGPIO_1, TerminalBlock_Phoenix:TerminalBlock_Phoenix_MKDS-1-6-3.81_1x06_P3.81mm_Horizontal, symbol Connector:Screw_Terminal_01x06
- added J5: FlexGPIO_2, TerminalBlock_Phoenix:TerminalBlock_Phoenix_MKDS-1-6-3.81_1x06_P3.81mm_Horizontal, symbol Connector:Screw_Terminal_01x06
Connections:
- net IN_FLOWMETER_GROUP_TWO is gone; now on net IN_FLOWMETER_GROUP_ONE: U1.6 (GPI35)
- net +5V: now also J1.2 (Pin_2)
- net FLEXIBLE_IO_01: now also J4.1 (Pin_1)
- net FLEXIBLE_IO_02: now also J4.2 (Pin_2)
- net FLEXIBLE_IO_03: now also J4.3 (Pin_3)
- net FLEXIBLE_IO_04: now also J4.4 (Pin_4)
- net FLEXIBLE_IO_05: now also J4.5 (Pin_5)
- net FLEXIBLE_IO_06: now also J4.6 (Pin_6)
- net FLEXIBLE_IO_07: now also J5.1 (Pin_1)
- net FLEXIBLE_IO_08: now also J5.2 (Pin_2)
- net FLEXIBLE_IO_09: now also J5.3 (Pin_3)
- net FLEXIBLE_IO_10: now also J5.4 (Pin_4)
- net FLEXIBLE_IO_11: now also J5.5 (Pin_5)
- net FLEXIBLE_IO_12: now also J5.6 (Pin_6)
- net GND: now also J1.1 (Pin_1), J2.1 (Pin_1), J3.1 (Pin_1)
- net IN_FLOWMETER_GROUP_ONE: now also J2.2 (Pin_2), J3.2 (Pin_2)
- net 3.3V renamed +3.3V
- net +3.3V: now also J2.3 (Pin_3), J3.3 (Pin_3)
Other:
- note removed: "TODO - Add pin here"

Commit message: some more pcb additions
Parts:
- added J10: Boiler Probe, TerminalBlock_Phoenix:TerminalBlock_Phoenix_MKDS-1-2-3.81_1x02_P3.81mm_Horizontal, symbol Connector:Screw_Terminal_01x02
- added J11: SOL_L_FUSE, new_local:696108003002, symbol new_local:696108003002
- added J12: 5V_FUSE, new_local:696108003002, symbol new_local:696108003002
- added J6: RelayOut_1, TerminalBlock_Phoenix:TerminalBlock_Phoenix_MKDS-1-4-3.81_1x04_P3.81mm_Horizontal, symbol Connector:Screw_Terminal_01x06
- added J7: RelayOut2, TerminalBlock_Phoenix:TerminalBlock_Phoenix_MKDS-1-4-3.81_1x04_P3.81mm_Horizontal, symbol Connector:Screw_Terminal_01x04
- added J8: Solenoid Power, TerminalBlock_Phoenix:TerminalBlock_Phoenix_MKDS-1-2-3.81_1x02_P3.81mm_Horizontal, symbol Connector:Screw_Terminal_01x02
- added J9: Pump Power, TerminalBlock_Phoenix:TerminalBlock_Phoenix_MKDS-1-2-3.81_1x02_P3.81mm_Horizontal, symbol Connector:Screw_Terminal_01x02
- added R5, R7: 10k, Resistor_THT:R_Axial_DIN0204_L3.6mm_D1.6mm_P2.54mm_Vertical, symbol Device:R
- added R8: R, Resistor_THT:R_Axial_DIN0207_L6.3mm_D2.5mm_P7.62mm_Horizontal, symbol Device:R
- K1, K2, K3, K4, K5: footprint G3MB-202P DC5_OMR -> new_local:G3MB-202P DC5_OMR
- U1: footprint esp32_lora_v2:esp32_devkitv4_38pin -> new_local:esp32_38pin
Connections:
- net +5V: now also J12.1, J12.2, R8.2
- net AC_PUMP_POWER_OUT: now also J7.2 (Pin_2)
- net AC_SOLENOID_BOILER_FILL: now also J7.4 (Pin_4)
- net AC_SOLENOID_GROUP_ONE: now also J6.6 (Pin_6)
- net AC_SOLENOID_GROUP_TWO: now also J6.4 (Pin_4)
- net AC_SOLENOID_TEA: now also J6.2 (Pin_2)
- net GND: now also J10.1 (Pin_1), R7.2
- net IN_BOILER_PROBE: now also J10.2 (Pin_2), R5.1, R7.1
- net IN_FLOWMETER_GROUP_ONE: now also R8.1
- net OUT_BOILER_PROBE_VOLTAGE: now also R5.2
- net AC_PUMP_POWER_IN renamed AC_PUMP_PHASE
- net AC_PUMP_PHASE: now also J9.2 (Pin_2)
- net AC_SOLENOID_INPUT_VOLTAGE renamed AC_SOLENOID_PHASE
- net AC_SOLENOID_PHASE: now also J11.2
- new net AC_PUMP_NEUTRAL: J7.1 (Pin_1), J9.1 (Pin_1)
- new net AC_SOLENOID_NEUTRAL: J6.1 (Pin_1), J6.3 (Pin_3), J6.5 (Pin_5), J7.3 (Pin_3), J8.1 (Pin_1)
- new net SOL_L: J11.1, J8.2 (Pin_2)
Other:
- moved on the sheet: J1

Commit message: implemented more fixes and initial clean routing pass of the pcb
Parts:
- added D1: PUMP_ON, LED_THT:LED_D3.0mm, symbol Device:LED
- added D2: BOILER_FILL_ON, LED_THT:LED_D3.0mm, symbol Device:LED
- added D3: GROUP1_ON, LED_THT:LED_D3.0mm, symbol Device:LED
- added D4: GROUP2_ON, LED_THT:LED_D3.0mm, symbol Device:LED
- added D5: TEA_ON, LED_THT:LED_D3.0mm, symbol Device:LED
- added R10, R11, R12, R13, R14: 1k, Resistor_THT:R_Axial_DIN0207_L6.3mm_D2.5mm_P7.62mm_Horizontal, symbol Device:R
- added R9: 10k, Resistor_THT:R_Axial_DIN0207_L6.3mm_D2.5mm_P7.62mm_Horizontal, symbol Device:R
- J10: Electrical_Rating (none) -> Boiler probe input: 0-5V nominal, 6.6V absolute max with 10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
- J11: Fuse_Rating (none) -> SOL_L common fuse holder: fit <=3A AC fuse, voltage/breakin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
- J12: Fuse_Rating (none) -> 5V fuse holder: fit <=1A fuse sized for ESP32 + SSR LED cur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
- J4, J5: Electrical_Rating (none) -> Flex IO: ESP32 3.3V GPIO only, 12mA max recommended per pin
- J6: footprint TerminalBlock_Phoenix:TerminalBlock_Phoenix_MKDS-1-4-3.81_1x04_P3.81mm_Horizontal -> TerminalBlock_Phoenix:TerminalBlock_Phoenix_MKDS-1-6-3.81_1x06_P3.81mm_Horizontal; Electrical_Rating (none) -> Solenoid outputs: 2A max per switched output; shared soleno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
- J7: Electrical_Rating (none) -> Pump output 2A max; boiler fill output 2A max; AC load only
- J8: Electrical_Rating (none) -> Solenoid AC input: shared bus 3A total continuous max, fuse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
- J9: Electrical_Rating (none) -> Pump AC input/output path: 2A max due G3MB SSR
- K1, K2, K3, K4, K5: Electrical_Rating (none) -> G3MB-202P DC5; output 2A max; 75-264VAC datasheet, 24VAC ou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
- R1, R2, R3, R4, R6: value R -> 4.7k
- R8: value R -> 10k
Connections:
- net +3.3V: now also R8.2, R9.2
- net +5V: now also R10.1, R11.1, R12.1, R13.1, R14.1; no longer R8.2
- net IN_FLOWMETER_GROUP_ONE: now also R9.1; no longer J3.2 (Pin_2), R8.1, U1.6 (GPI35)
- new net IN_FLOWMETER_GROUP_TWO: J3.2 (Pin_2), R8.1, U1.6 (GPI35)
- new net LED_BOILER_FILL_A: D2.2 (A), R11.2
- new net LED_GROUP1_A: D3.2 (A), R12.2
- new net LED_GROUP2_A: D4.2 (A), R13.2
- new net LED_PUMP_A: D1.2 (A), R10.2
- new net LED_TEA_A: D5.2 (A), R14.2
- new net Net-(Q1-C): D1.1 (K)
- new net Net-(Q2-C): D2.1 (K)
- new net Net-(Q3-C): D3.1 (K)
- new net Net-(Q4-C): D4.1 (K)
- new net Net-(Q5-C): D5.1 (K)
- no-connect marks 0 -> 13
Other:
- note added: "DESIGN RATINGS / LIMITS AC outputs use G3MB-202P DC5 SSRs: 2 A max per output, AC load only. Datasheet load range is 75-264 VAC; 24 VAC use is intentionally out-of-datasheet/prototype-only. Board current assumption: 1 oz copper, 1.5 mm AC tracks. Limit shared solenoid common bus to 3 A total continuous; each switched output and pump output to 2 A max. Fusing required: SOL_L common fuse <= 3 A, ea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"

Commit message: pcb updates
Parts:
- added C1, C2: 1nF, Capacitor_THT:C_Disc_D5.0mm_W2.5mm_P5.00mm, symbol Device:C
- added C3: 100nF, Capacitor_THT:C_Disc_D5.0mm_W2.5mm_P5.00mm, symbol Device:C
- added D6, D7, D8: PESD3V3, Diode_THT:D_DO-35_SOD27_P7.62mm_Horizontal, symbol Device:D_Zener
- J12: value 5V_FUSE -> 5V_FUSE_5x20mm; footprint new_local:696108003002 -> Fuse:Fuseholder_Cylinder-5x20mm_Schurter_0031_8201_Horizontal_Open; Fuse_Rating 5V fuse holder: fit <=1A fuse sized for ESP32 + SSR LED cur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 -> 5x20 mm glass/cartridge fuse holder: fit <=1A fuse sized fo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
Connections:
- net +5V: no longer J1.2 (Pin_2), J12.1
- net GND: now also U1.14 (GND), U1.32 (GND), C1.2, C2.2, C3.2, D6.2 (A), D7.2 (A), D8.2 (A)
- net IN_BOILER_PROBE: now also C3.1, D8.1 (K)
- net IN_FLOWMETER_GROUP_ONE: now also C1.1, D6.1 (K)
- net IN_FLOWMETER_GROUP_TWO: now also C2.1, D7.1 (K)
- new net 5V_RAW: J1.2 (Pin_2), J12.1
- no-connect marks 13 -> 11
Other:
- note added: "DESIGN RATINGS / LIMITS AC outputs use G3MB-202P DC5 SSRs: 2 A max per output, AC load only. Datasheet load range is 75-264 VAC; 24 VAC use is intentionally out-of-datasheet/prototype-only. Board current assumption: 1 oz copper, 2.0 mm AC tracks. Limit shared solenoid common bus to 3 A total continuous; each switched output and pump output to 2 A max. Fusing required: SOL_L common fuse <= 3 A, ea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"
- note removed: "DESIGN RATINGS / LIMITS AC outputs use G3MB-202P DC5 SSRs: 2 A max per output, AC load only. Datasheet load range is 75-264 VAC; 24 VAC use is intentionally out-of-datasheet/prototype-only. Board current assumption: 1 oz copper, 1.5 mm AC tracks. Limit shared solenoid common bus to 3 A total continuous; each switched output and pump output to 2 A max. Fusing required: SOL_L common fuse <= 3 A, ea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"
