File: pcb/BrewPilot.kicad_sch (KiCad schematic)
At the start: 48 parts, among them J1 5V Power, J10 Boiler Probe, J11 SOL_L_FUSE, J12 5V_FUSE_5x20mm, J2 Flow Meter Group One, J3 Flow Meter Group Two, J4 FlexGPIO_1, J5 FlexGPIO_2, J6 RelayOut_1, J7 RelayOut2, J8 Solenoid Power, J9 Pump Power, K1 G3MB-202P DC5, K2 G3MB-202P DC5, K3 G3MB-202P DC5, K4 G3MB-202P DC5, K5 G3MB-202P DC5, Q1 BC547, Q2 BC547, Q3 BC547, Q4 BC547, Q5 BC547, U1 esp32

Commit message: stash
Parts:
- added C4: 100uF, Capacitor_THT:CP_Radial_D6.3mm_P2.50mm, symbol Device:C_Polarized
- added C5: 100nF, Capacitor_THT:C_Disc_D5.0mm_W2.5mm_P5.00mm, symbol Device:C
- added J13: I2C Port, Connector_RJ:RJ45_Amphenol_54602-x08_Horizontal, symbol Connector:8P8C
- added R15, R16: 4.7k, Resistor_THT:R_Axial_DIN0207_L6.3mm_D2.5mm_P7.62mm_Horizontal, symbol Device:R
Connections:
- net +3.3V: now also J13.4, R15.1, R16.1
- net +5V: now also C4.1, C5.1
- net CONTROL_RELAY_BOILER_FILL: now also U1.30 (GPIO18); no longer U1.24 (GPIO2)
- net CONTROL_RELAY_GROUP_ONE: now also U1.26 (GPIO4); no longer U1.29 (GPIO5)
- net CONTROL_RELAY_GROUP_TWO: now also U1.24 (GPIO2); no longer U1.26 (GPIO4)
- net CONTROL_RELAY_PUMP: now also U1.29 (GPIO5); no longer U1.30 (GPIO18)
- net FLEXIBLE_IO_10: now also J13.1, R15.2
- net FLEXIBLE_IO_11: now also J13.2, R16.2
- net GND: now also C4.2, C5.2, J13.3, J13.5, J13.6, J13.7, J13.8

Commit message: cleanup and first pcb order
Parts:
- D6, D7, D8: value PESD3V3 -> BZX55C5V1
Connections:
- net Net-(Q1-C) is gone; now on net SSR_PUMP_SINK: D1.1 (K)
- net Net-(Q2-C) is gone; now on net SSR_BOILER_FILL_SINK: D2.1 (K)
- net Net-(Q3-C) is gone; now on net SSR_GROUP1_SINK: D3.1 (K)
- net Net-(Q4-C) is gone; now on net SSR_GROUP2_SINK: D4.1 (K)
- net Net-(Q5-C) is gone; now on net SSR_TEA_SINK: D5.1 (K)
- net SSR_BOILER_FILL_SINK: now reaches K2.4, Q2.1 (C)
- net SSR_GROUP2_SINK: now reaches K4.4, Q4.1 (C)
- net SSR_GROUP1_SINK: now reaches K3.4, Q3.1 (C)
- net SSR_TEA_SINK: now reaches K5.4, Q5.1 (C)
- net SSR_PUMP_SINK: now reaches K1.4, Q1.1 (C)

Commit message: Save current BrewPilot PCB design before schematic alignment
Amp-Thread-ID: https://ampcode.com/threads/T-01a0debc-596d-7434-9824-16fe8385066c
Co-authored-by: Amp <amp@ampcode.com>
Parts:
- J11: footprint new_local:696108003002 -> new_local:BLX-A_5x20mm
- J12: footprint Fuse:Fuseholder_Cylinder-5x20mm_Schurter_0031_8201_Horizontal_Open -> new_local:BLX-A_5x20mm
- Q1, Q2, Q3, Q4, Q5: footprint Package_TO_SOT_THT:TO-92_Inline -> Package_TO_SOT_THT:TO-92_Inline_Wide
Changed lines of the file:
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@@
 			)
 		)
-		(property "Footprint" "Package_TO_SOT_THT:TO-92_Inline"
+		(property "Footprint" "Package_TO_SOT_THT:TO-92_Inline_Wide"
 			(at 262.255 49.53 0)
 			(effects
@@
 			)
 		)
-		(property "Footprint" "Package_TO_SOT_THT:TO-92_Inline"
+		(property "Footprint" "Package_TO_SOT_THT:TO-92_Inline_Wide"
 			(at 262.255 100.33 0)
 			(effects
@@
 			)
 		)
-		(property "Footprint" "Package_TO_SOT_THT:TO-92_Inline"
+		(property "Footprint" "Package_TO_SOT_THT:TO-92_Inline_Wide"
 			(at 262.255 74.93 0)
 			(effects
@@
 			)
 		)
-		(property "Footprint" "new_local:696108003002"
+		(property "Footprint" "new_local:BLX-A_5x20mm"
 			(at 33.02 134.62 0)
 			(effects
@@
 			)
 		)
-		(property "Footprint" "Package_TO_SOT_THT:TO-92_Inline"
+		(property "Footprint" "Package_TO_SOT_THT:TO-92_Inline_Wide"
 			(at 262.255 125.73 0)
 			(effects
@@
 			)
 		)
-		(property "Footprint" "Fuse:Fuseholder_Cylinder-5x20mm_Schurter_0031_8201_Horizontal_Open"
+		(property "Footprint" "new_local:BLX-A_5x20mm"
 			(at 41.91 121.92 0)
 			(effects
@@
 			)
 		)
-		(property "Footprint" "Package_TO_SOT_THT:TO-92_Inline"
+		(property "Footprint" "Package_TO_SOT_THT:TO-92_Inline_Wide"
 			(at 262.255 24.13 0)
 			(effects

Commit message: ai driven improvements
Parts:
- J10: Electrical_Rating Boiler probe input: 0-5V nominal, 6.6V absolute max with 10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 -> Boiler probe connects directly to GPIO34 ADC; no 5V-toleran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
- R5, R7: footprint Resistor_THT:R_Axial_DIN0204_L3.6mm_D1.6mm_P2.54mm_Vertical -> Resistor_THT:R_Axial_DIN0207_L6.3mm_D2.5mm_P7.62mm_Horizontal
Other:
- note added: "DESIGN LIMITS - NOT MAINS-CERTIFIED G3MB-202P DC5: AC loads only, 2 A max each; 75-264 VAC per datasheet. 24 VAC is outside the specified load range. Assume 1 oz copper and 2 mm AC tracks. Shared solenoid bus: 3 A total continuous; individual outputs: 2 A max. Fit SOL_L fuse <= 3 A and 5 V fuse <= 1 A. Protect each load's wiring externally; select fuse breaking capacity. PCB rule: 6 mm AC-to-low-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"
- note removed: "DESIGN RATINGS / LIMITS AC outputs use G3MB-202P DC5 SSRs: 2 A max per output, AC load only. Datasheet load range is 75-264 VAC; 24 VAC use is intentionally out-of-datasheet/prototype-only. Board current assumption: 1 oz copper, 2.0 mm AC tracks. Limit shared solenoid common bus to 3 A total continuous; each switched output and pump output to 2 A max. Fusing required: SOL_L common fuse <= 3 A, ea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"
- moved on the sheet: C1, C2, C3, C4, C5, D1, D2, D3, D4, D5, D6, D7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
