File: pcb/BrewPilot.kicad_sch (KiCad schematic)
At the start: 53 parts, among them J1 5V Power, J10 Boiler Probe, J11 SOL_L_FUSE, J12 5V_FUSE_5x20mm, J13 I2C Port, J2 Flow Meter Group One, J3 Flow Meter Group Two, J4 FlexGPIO_1, J5 FlexGPIO_2, J6 RelayOut_1, J7 RelayOut2, J8 Solenoid Power, J9 Pump Power, K1 G3MB-202P DC5, K2 G3MB-202P DC5, K3 G3MB-202P DC5, K4 G3MB-202P DC5, K5 G3MB-202P DC5, Q1 BC547, Q2 BC547, Q3 BC547, Q4 BC547, Q5 BC547, U1 esp32

Commit message: Checkpoint current PCB revision and machine-specific firmware builds
Preserve the existing workspace before firmware safety fixes.

Amp-Thread-ID: https://ampcode.com/threads/T-01a12a1e-8ea4-702d-96da-3a9264193d9b
Co-authored-by: Amp <amp@ampcode.com>
Parts:
- added R17, R18, R19, R20, R21: 4.7k, Resistor_THT:R_Axial_DIN0207_L6.3mm_D2.5mm_P7.62mm_Horizontal, symbol Device:R
- added R22, R23, R24, R25, R26, R27: 10k, Resistor_THT:R_Axial_DIN0207_L6.3mm_D2.5mm_P7.62mm_Horizontal, symbol Device:R
- J13: footprint Connector_RJ:RJ45_Amphenol_54602-x08_Horizontal -> new_local:RJ45_Amphenol_54602-x08_BoardEdge
Connections:
- net +3.3V: now also R22.1, R23.1, R24.1, R25.1, R26.1, R27.1
- net FLEXIBLE_IO_01: now also U1.3 (GPI36), R22.2; no longer U1.15 (GPIO13)
- net FLEXIBLE_IO_03: now also U1.4 (GPI39), R23.2; no longer U1.12 (GPIO14)
- net FLEXIBLE_IO_04: now also R27.2
- net FLEXIBLE_IO_05: now also R26.2
- net FLEXIBLE_IO_06: now also R25.2
- net FLEXIBLE_IO_10: now also U1.15 (GPIO13); no longer J13.1, R15.2, U1.33 (GPIO21)
- net FLEXIBLE_IO_11: now also U1.12 (GPIO14); no longer J13.2, R16.2, U1.36 (GPIO22)
- net FLEXIBLE_IO_12: now also R24.2
- net GND: now also R17.2, R18.2, R19.2, R20.2, R21.2
- net at Q3.2 (B), R2.2: now also R19.1
- net at Q2.2 (B), R1.1: now also R18.1
- net at Q4.2 (B), R3.1: now also R20.1
- net at Q5.2 (B), R4.1: now also R21.1
- net at Q1.2 (B), R6.1: now also R17.1
- new net I2C_SCL: J13.2, R16.2, U1.36 (GPIO22)
- new net I2C_SDA: J13.1, R15.2, U1.33 (GPIO21)
- no-connect marks 11 -> 9
