File: pcb/BrewPilot.kicad_sch (KiCad schematic)
At the start: 19 parts, among them K1 G3MB-202P DC5, K2 G3MB-202P DC5, K3 G3MB-202P DC5, K4 G3MB-202P DC5, K5 G3MB-202P DC5, K6 G3MB-202P DC5, Q1 BC547, Q2 BC547, Q3 BC547, Q4 BC547, Q5 BC547, Q6 BC547, U1 esp32

Commit message: Integrate compact PCB revision with matching machine pin firmware
Amp-Thread-ID: https://ampcode.com/threads/T-01a12f6a-38bb-752f-a21e-c225bfa986bd
Parts:
- removed K6: G3MB-202P DC5, G3MB-202P DC5_OMR, symbol new_local:G3MB-202P_DC5
- removed Q6: BC547, Package_TO_SOT_THT:TO-92_Inline, symbol Transistor_BJT:BC547
- added C1, C2: 1nF, Capacitor_THT:C_Disc_D5.0mm_W2.5mm_P5.00mm, symbol Device:C
- added C3, C5: 100nF, Capacitor_THT:C_Disc_D5.0mm_W2.5mm_P5.00mm, symbol Device:C
- added C4: 100uF, Capacitor_THT:CP_Radial_D6.3mm_P2.50mm, symbol Device:C_Polarized
- added D1: PUMP_ON, LED_THT:LED_D3.0mm, symbol Device:LED
- added D2: BOILER_FILL_ON, LED_THT:LED_D3.0mm, symbol Device:LED
- added D3: GROUP1_ON, LED_THT:LED_D3.0mm, symbol Device:LED
- added D4: GROUP2_ON, LED_THT:LED_D3.0mm, symbol Device:LED
- added D5: TEA_ON, LED_THT:LED_D3.0mm, symbol Device:LED
- added D6, D7, D8: BZX55C5V1, Diode_THT:D_DO-35_SOD27_P7.62mm_Horizontal, symbol Device:D_Zener
- added J1: 5V Power, TerminalBlock_Phoenix:TerminalBlock_Phoenix_MKDS-1-2-3.81_1x02_P3.81mm_Horizontal, symbol Connector:Screw_Terminal_01x02
- added J10: Boiler Probe, TerminalBlock_Phoenix:TerminalBlock_Phoenix_MKDS-1-2-3.81_1x02_P3.81mm_Horizontal, symbol Connector:Screw_Terminal_01x02
- added J11: SOL_L_FUSE, new_local:BLX-A_5x20mm, symbol new_local:696108003002
- added J12: 5V_FUSE_5x20mm, new_local:BLX-A_5x20mm, symbol new_local:696108003002
- added J13: I2C Port, new_local:RJ45_Amphenol_54602-x08_BoardEdge, symbol Connector:8P8C
- added J2: Flow Meter Group One, TerminalBlock_Phoenix:TerminalBlock_Phoenix_MKDS-1-3-3.81_1x03_P3.81mm_Horizontal, symbol Connector:Screw_Terminal_01x03
- added J3: Flow Meter Group Two, TerminalBlock_Phoenix:TerminalBlock_Phoenix_MKDS-1-3-3.81_1x03_P3.81mm_Horizontal, symbol Connector:Screw_Terminal_01x03
- added J4: FlexGPIO_1, TerminalBlock_Phoenix:TerminalBlock_Phoenix_MKDS-1-6-3.81_1x06_P3.81mm_Horizontal, symbol Connector:Screw_Terminal_01x06
- added J5: FlexGPIO_2, TerminalBlock_Phoenix:TerminalBlock_Phoenix_MKDS-1-6-3.81_1x06_P3.81mm_Horizontal, symbol Connector:Screw_Terminal_01x06
- added J6: RelayOut_1, TerminalBlock_Phoenix:TerminalBlock_Phoenix_MKDS-1-6-3.81_1x06_P3.81mm_Horizontal, symbol Connector:Screw_Terminal_01x06
- added J7: RelayOut2, TerminalBlock_Phoenix:TerminalBlock_Phoenix_MKDS-1-4-3.81_1x04_P3.81mm_Horizontal, symbol Connector:Screw_Terminal_01x04
- added J8: Solenoid Power, TerminalBlock_Phoenix:TerminalBlock_Phoenix_MKDS-1-2-3.81_1x02_P3.81mm_Horizontal, symbol Connector:Screw_Terminal_01x02
- added J9: Pump Power, TerminalBlock_Phoenix:TerminalBlock_Phoenix_MKDS-1-2-3.81_1x02_P3.81mm_Horizontal, symbol Connector:Screw_Terminal_01x02
- added R10, R11, R12, R13, R14: 1k, Resistor_THT:R_Axial_DIN0207_L6.3mm_D2.5mm_P7.62mm_Horizontal, symbol Device:R
- added R15, R16, R17, R18, R19, R20, R21: 4.7k, Resistor_THT:R_Axial_DIN0207_L6.3mm_D2.5mm_P7.62mm_Horizontal, symbol Device:R
- added R22, R23, R24, R25, R26, R27, R7, R8, R9: 10k, Resistor_THT:R_Axial_DIN0207_L6.3mm_D2.5mm_P7.62mm_Horizontal, symbol Device:R
- K1, K2, K3, K4, K5: footprint G3MB-202P DC5_OMR -> new_local:G3MB-202P DC5_OMR; Electrical_Rating (none) -> G3MB-202P DC5; output 2A max; 75-264VAC datasheet, 24VAC ou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
- Q1, Q2, Q3, Q4, Q5: footprint Package_TO_SOT_THT:TO-92_Inline -> Package_TO_SOT_THT:TO-92_Inline_Wide
- R1, R2, R3, R4, R6: value R -> 4.7k
- R5: value R -> 10k
- U1: footprint esp32_lora_v2:esp32_devkitv4_38pin -> new_local:esp32_38pin
Connections:
- net +5V: now also C4.1, C5.1, J12.2, R10.1, R11.1, R12.1, R13.1, R14.1
- net AC_PUMP_POWER_OUT: now also J7.2 (Pin_2)
- net AC_SOLENOID_BOILER_FILL: now also J7.4 (Pin_4)
- net AC_SOLENOID_GROUP_ONE: now also J6.6 (Pin_6)
- net AC_SOLENOID_GROUP_TWO: now also J6.4 (Pin_4)
- net AC_SOLENOID_TEA: now also J6.2 (Pin_2)
- net CONTROL_RELAY_BOILER_FILL: now also U1.30 (GPIO18); no longer U1.24 (GPIO2)
- net CONTROL_RELAY_GROUP_ONE: now also U1.26 (GPIO4); no longer U1.29 (GPIO5)
- net CONTROL_RELAY_GROUP_TWO: now also U1.24 (GPIO2); no longer U1.26 (GPIO4)
- net CONTROL_RELAY_PUMP: now also U1.29 (GPIO5); no longer U1.30 (GPIO18)
- net FLEXIBLE_IO_01: now also U1.3 (GPI36), J4.1 (Pin_1), R22.2; no longer U1.15 (GPIO13)
- net FLEXIBLE_IO_02: now also J4.2 (Pin_2)
- net FLEXIBLE_IO_03: now also U1.4 (GPI39), J4.3 (Pin_3), R23.2; no longer U1.12 (GPIO14)
- net FLEXIBLE_IO_04: now also J4.4 (Pin_4), R27.2
- net FLEXIBLE_IO_05: now also J4.5 (Pin_5), R26.2
- net FLEXIBLE_IO_06: now also J4.6 (Pin_6), R25.2
- net FLEXIBLE_IO_07: now also J5.1 (Pin_1)
- net FLEXIBLE_IO_08: now also J5.2 (Pin_2)
- net FLEXIBLE_IO_09: now also J5.3 (Pin_3)
- net FLEXIBLE_IO_10: now also U1.15 (GPIO13), J5.4 (Pin_4); no longer U1.33 (GPIO21)
- net FLEXIBLE_IO_11: now also U1.12 (GPIO14), J5.5 (Pin_5); no longer U1.36 (GPIO22)
- net FLEXIBLE_IO_12: now also J5.6 (Pin_6), R24.2
- net GND: now also U1.14 (GND), U1.32 (GND), C1.2, C2.2, C3.2, C4.2, C5.2, D6.2 (A), D7.2 (A), D8.2 (A), J1.1 (Pin_1), J10.1 (Pin_1), J13.3, J13.5, J13.6, J13.7, J13.8, J2.1 (Pin_1), J3.1 (Pin_1), R17.2, R18.2, R19.2, R20.2, R21.2, R7.2
- net IN_BOILER_PROBE: now also R5.1, C3.1, D8.1 (K), J10.2 (Pin_2), R7.1
- net IN_FLOWMETER_GROUP_ONE: now also C1.1, D6.1 (K), J2.2 (Pin_2), R9.1
- net IN_FLOWMETER_GROUP_TWO: now also C2.1, D7.1 (K), J3.2 (Pin_2), R8.1
- net OUT_BOILER_PROBE_VOLTAGE: now also R5.2
- net at Q3.2 (B), R2.2: now also R19.1
- net SSR_BOILER_FILL_SINK: now reaches K2.4, Q2.1 (C)
- net SSR_BOILER_FILL_SINK: now also D2.1 (K)
- net at Q2.2 (B), R1.1: now also R18.1
- net SSR_GROUP2_SINK: now reaches K4.4, Q4.1 (C)
- net SSR_GROUP2_SINK: now also D4.1 (K)
- net at Q4.2 (B), R3.1: now also R20.1
- net SSR_GROUP1_SINK: now reaches K3.4, Q3.1 (C)
- net SSR_GROUP1_SINK: now also D3.1 (K)
- net SSR_TEA_SINK: now reaches K5.4, Q5.1 (C)
- net SSR_TEA_SINK: now also D5.1 (K)
- net at Q5.2 (B), R4.1: now also R21.1
- net SSR_PUMP_SINK: now reaches K1.4, Q1.1 (C)
- net SSR_PUMP_SINK: now also D1.1 (K)
- net at Q1.2 (B), R6.1: now also R17.1
- net 3.3V renamed +3.3V
- net +3.3V: now also J13.4, J2.3 (Pin_3), J3.3 (Pin_3), R15.1, R16.1, R22.1, R23.1, R24.1, R25.1, R26.1, R27.1, R8.2, R9.2
- net AC_PUMP_POWER_IN renamed AC_PUMP_PHASE
- net AC_PUMP_PHASE: now also J9.2 (Pin_2)
- net AC_SOLENOID_INPUT_VOLTAGE renamed AC_SOLENOID_PHASE
- net AC_SOLENOID_PHASE: now also J11.2
- new net 5V_RAW: J1.2 (Pin_2), J12.1
- new net AC_PUMP_NEUTRAL: J7.1 (Pin_1), J9.1 (Pin_1)
- new net AC_SOLENOID_NEUTRAL: J6.1 (Pin_1), J6.3 (Pin_3), J6.5 (Pin_5), J7.3 (Pin_3), J8.1 (Pin_1)
- new net I2C_SCL: J13.2, R16.2, U1.36 (GPIO22)
- new net I2C_SDA: J13.1, R15.2, U1.33 (GPIO21)
- new net LED_BOILER_FILL_A: D2.2 (A), R11.2
- new net LED_GROUP1_A: D3.2 (A), R12.2
- new net LED_GROUP2_A: D4.2 (A), R13.2
- new net LED_PUMP_A: D1.2 (A), R10.2
- new net LED_TEA_A: D5.2 (A), R14.2
- new net SOL_L: J11.1, J8.2 (Pin_2)
- no-connect marks 0 -> 9
Other:
- note added: "DESIGN LIMITS - NOT MAINS-CERTIFIED G3MB-202P DC5: AC loads only, 2 A max each; 75-264 VAC per datasheet. 24 VAC is outside the specified load range. Assume 1 oz copper and 2 mm AC tracks. Shared solenoid bus: 3 A total continuous; individual outputs: 2 A max. Fit SOL_L fuse <= 3 A and 5 V fuse <= 1 A. Protect each load's wiring externally; select fuse breaking capacity. PCB rule: 6 mm AC-to-low-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"
- note removed: "TODO - Add pin here"
- moved on the sheet: K1, K2, K3, K4, K5, Q1, Q2, Q3, Q4, Q5, R1, R2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
