File: pcb/BrewPilot.kicad_pcb (KiCad board)
At the start: 2 copper layers, 147.5 x 129 mm, 48 parts, among them J1 5V Power, J10 Boiler Probe, J11 SOL_L_FUSE, J12 5V_FUSE_5x20mm, J2 Flow Meter Group One, J3 Flow Meter Group Two, J4 FlexGPIO_1, J5 FlexGPIO_2, J6 RelayOut_1, J7 RelayOut2, J8 Solenoid Power, J9 Pump Power, K1 G3MB-202P DC5, K2 G3MB-202P DC5, K3 G3MB-202P DC5, K4 G3MB-202P DC5, K5 G3MB-202P DC5, Q1 BC547, Q2 BC547, Q3 BC547, Q4 BC547, Q5 BC547, U1 esp32

Commit message: stash
Parts:
- added C4: 100uF, Capacitor_THT:CP_Radial_D6.3mm_P2.50mm, F.Cu at (133.0, 82.9)
- added C5: 100nF, Capacitor_THT:C_Disc_D5.0mm_W2.5mm_P5.00mm, F.Cu at (124.0, 84.4)
- added H1: MountingHole_3.2mm_M3, MountingHole_3.2mm_M3, F.Cu at (119.5, 39.5)
- added H2: MountingHole_3.2mm_M3, MountingHole_3.2mm_M3, F.Cu at (226.0, 50.5)
- added H3: MountingHole_3.2mm_M3, MountingHole_3.2mm_M3, F.Cu at (121.0, 161.5)
- added H4: MountingHole_3.2mm_M3, MountingHole_3.2mm_M3, F.Cu at (226.0, 161.5)
- added J13: I2C Port, Connector_RJ:RJ45_Amphenol_54602-x08_Horizontal, F.Cu at (141.1, 106.7)
- added R15: 4.7k, Resistor_THT:R_Axial_DIN0207_L6.3mm_D2.5mm_P7.62mm_Horizontal, F.Cu at (160.0, 59.5)
- added R16: 4.7k, Resistor_THT:R_Axial_DIN0207_L6.3mm_D2.5mm_P7.62mm_Horizontal, F.Cu at (160.0, 54.5)
- moved J1 139.3 mm to (129.6, 42.9), turned to 180 degrees
- moved R11 137.1 mm to (218.6, 75.3), turned to -90 degrees
- moved R10 124.5 mm to (208.1, 75.6), turned to -90 degrees
- moved R12 121.8 mm to (198.5, 75.5), turned to -90 degrees
- moved D2 118.2 mm to (218.6, 90.3), turned to -90 degrees
- moved R13 116.8 mm to (188.0, 75.2), turned to -90 degrees
- moved R14 112.9 mm to (177.5, 75.2), turned to -90 degrees
- moved D1 105.9 mm to (208.1, 90.6), turned to -90 degrees
- moved D3 101.8 mm to (198.5, 90.5), turned to -90 degrees
- moved D4 96.1 mm to (188.0, 90.2), turned to -90 degrees
- moved D5 91.9 mm to (177.5, 90.2), turned to -90 degrees
- moved J12 83.5 mm to (128.8, 62.9), turned to -90 degrees
- moved U1 80.0 mm to (156.1, 50.2), turned to 0 degrees
- moved R7 57.9 mm to (189.5, 62.0), turned to -90 degrees
- moved D8 52.0 mm to (181.9, 51.5)
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Connections:
- U1 pad 24: CONTROL_RELAY_BOILER_FILL -> CONTROL_RELAY_GROUP_TWO
- U1 pad 26: CONTROL_RELAY_GROUP_TWO -> CONTROL_RELAY_GROUP_ONE
- U1 pad 29: CONTROL_RELAY_GROUP_ONE -> CONTROL_RELAY_PUMP
- U1 pad 30: CONTROL_RELAY_PUMP -> CONTROL_RELAY_BOILER_FILL
Routing:
- net GND: track 298.4 -> 0.00 mm, vias 2 -> 0
- net CONTROL_RELAY_PUMP: track 146.7 -> 48.8 mm
- net Net-(Q1-C): track 128.8 -> 37.2 mm, vias 2 -> 0
- net Net-(Q2-C): track 115.8 -> 36.1 mm, vias 1 -> 0
- net AC_SOLENOID_GROUP_ONE: track 95.6 -> 27.8 mm
- net 5V_RAW: track 76.7 -> 9.92 mm
- net FLEXIBLE_IO_10: track 50.4 -> 115.2 mm
- net CONTROL_RELAY_BOILER_FILL: track 122.7 -> 59.8 mm
- net 5V: track 280.2 -> 223.1 mm, vias 2 -> 0
- net FLEXIBLE_IO_11: track 43.4 -> 99.9 mm
- net 3.3V: track 155.2 -> 211.7 mm, vias 0 -> 2
- net Net-(Q4-C): track 90.6 -> 36.3 mm, vias 1 -> 0
- net OUT_BOILER_PROBE_VOLTAGE: track 66.0 -> 18.2 mm
- net Net-(Q3-C): track 84.5 -> 37.2 mm, vias 1 -> 0
- net IN_FLOWMETER_GROUP_ONE: track 105.3 -> 58.5 mm
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- removed copper zone on F.Cu, net GND
Other:
- board size 147.5 x 129 mm -> 113 x 129 mm
- board text added: "+5V"
- board text added: "1 GND"
- board text added: "1 IO1"
- board text added: "1 IO10"
- board text added: "1 IO7"
- board text added: "1 N"
- board text added: "1 PN"
- board text added: "1 RAW"
- board text added: "1 SOL-L"
- board text added: "2 +5V"
- board text added: "2 AC-L"
- board text added: "2 IO11"
- board text added: "2 IO2"
- board text added: "2 IO8"
- board text added: "2 L"
- board text added: "2 PUMP"
- board text added: "2 SIG"
- board text added: "2 SOL-L"
- board text added: "2 TEA"
- board text added: "3 3V3"
- board text added: "3 GND"
- board text added: "3 IO3"
- board text added: "3 IO9"
- board text added: "3 N"
- board text added: "4 3V3"
- board text added: "4 FILL"
- board text added: "4 G2"
- board text added: "4 IO10"
- board text added: "4 IO4"
- board text added: "5 GND"
- board text added: "5 IO5"
- board text added: "5 N"
- board text added: "6 G1"
- board text added: "6 GND"
- board text added: "6 IO6"
- board text added: "7 GND"
- board text added: "8 GND"
- board text added: "C1 1n G1"
- board text added: "C2 1n G2"
- board text added: "C3 100n BP"
- board text added: "C4 100u"
- board text added: "C5 100n"
- board text added: "D1 PUMP"
- board text added: "D2 FILL"
- board text added: "D3 G1"
- board text added: "D4 G2"
- board text added: "D5 TEA"
- board text added: "D6 ESD G1"
- board text added: "D7 ESD G2"
- board text added: "D8 ESD BP"
- board text added: "GND"
- board text added: "H1 M3"
- board text added: "H2 M3"
- board text added: "H3 M3"
- board text added: "H4 M3"
- board text added: "IO11"
- board text added: "IO12"
- board text added: "J1 5V IN"
- board text added: "J10 BOILER"
- board text added: "J11 SOL FUSE"
- board text added: "J12 5V FUSE"
- board text added: "J13 I2C"
- board text added: "J2 FLOW1"
- board text added: "J3 FLOW2"
- board text added: "J4 IO1-6"
- board text added: "J5 IO7-12"
- board text added: "J6 SOL OUT"
- board text added: "J7 PUMP/FILL"
- board text added: "J8 SOL PWR"
- board text added: "J9 PUMP PWR"
- board text added: "K1 PUMP"
- board text added: "K2 FILL"
- board text added: "K3 G1"
- board text added: "K4 G2"
- board text added: "K5 TEA"
- board text added: "Q1 PUMP"
- board text added: "Q2 FILL"
- board text added: "Q3 G1"
- board text added: "Q4 G2"
- board text added: "Q5 TEA"
- board text added: "R1 4k7 FILL"
- board text added: "R10 1k PUMP"
- board text added: "R11 1k FILL"
- board text added: "R12 1k G1"
- board text added: "R13 1k G2"
- board text added: "R14 1k TEA"
- board text added: "R15 4k7 IO10"
- board text added: "R16 4k7 IO11"
- board text added: "R2 4k7 G1"
- board text added: "R3 4k7 G2"
- board text added: "R4 4k7 TEA"
- board text added: "R5 10k BP"
- board text added: "R6 4k7 PUMP"
- board text added: "R7 10k BP"
- board text added: "R8 10k FM2"
- board text added: "R9 10k FM1"
- board text added: "U1 ESP32"
- board text removed: "5V FUSE"
- board text removed: "5V IN"
- board text removed: "FILL"
- board text removed: "FLEX 1"
- board text removed: "FLEX 2"
- board text removed: "FLOW 1"
- board text removed: "FLOW 2"
- board text removed: "G1"
- board text removed: "G2"
- board text removed: "PROBE"
- board text removed: "PUMP"
- board text removed: "PUMP PWR"
- board text removed: "PUMP/SOL"
- board text removed: "SOL FUSE"
- board text removed: "SOL OUT"
- board text removed: "SOL PWR"
- board text removed: "TEA"

Commit message: cleanup and first pcb order
Parts:
- D6, D7, D8: value PESD3V3 -> BZX55C5V1
Connections:
- net 3.3V renamed +3.3V
- net 5V renamed +5V
- net Net-(Q1-C) renamed SSR_PUMP_SINK
- net Net-(Q2-C) renamed SSR_BOILER_FILL_SINK
- net Net-(Q3-C) renamed SSR_GROUP1_SINK
- net Net-(Q4-C) renamed SSR_GROUP2_SINK
- net Net-(Q5-C) renamed SSR_TEA_SINK
