File: pcb/BrewPilot.kicad_pcb (KiCad board)
At the start: 2 copper layers, 113 x 129 mm, 57 parts, among them J1 5V Power, J10 Boiler Probe, J11 SOL_L_FUSE, J12 5V_FUSE_5x20mm, J13 I2C Port, J2 Flow Meter Group One, J3 Flow Meter Group Two, J4 FlexGPIO_1, J5 FlexGPIO_2, J6 RelayOut_1, J7 RelayOut2, J8 Solenoid Power, J9 Pump Power, K1 G3MB-202P DC5, K2 G3MB-202P DC5, K3 G3MB-202P DC5, K4 G3MB-202P DC5, K5 G3MB-202P DC5, Q1 BC547, Q2 BC547, Q3 BC547, Q4 BC547, Q5 BC547, U1 esp32

Commit message: made pcb layout more compact
Parts:
- R5, R7: footprint Resistor_THT:R_Axial_DIN0204_L3.6mm_D1.6mm_P2.54mm_Vertical -> Resistor_THT:R_Axial_DIN0207_L6.3mm_D2.5mm_P7.62mm_Horizontal
- moved J13 47.6 mm to (151.5, 60.2)
- moved C5 45.0 mm to (166.0, 100.5)
- moved J12 44.4 mm to (167.0, 85.5), turned to 0 degrees
- moved J1 44.1 mm to (148.0, 83.0), turned to -90 degrees
- moved D8 43.1 mm to (209.2, 84.8), turned to 90 degrees
- moved R5 41.1 mm to (219.6, 83.0), turned to 0 degrees
- moved C3 40.7 mm to (214.7, 83.2), turned to 90 degrees
- moved R7 33.2 mm to (219.4, 76.5), turned to 0 degrees
- moved J11 31.5 mm to (175.0, 138.0)
- moved H1 31.3 mm to (148.0, 52.5)
- moved H3 30.6 mm to (151.5, 159.5)
- moved C4 30.4 mm to (158.5, 99.5)
- moved D6 18.1 mm to (207.7, 65.3), turned to 90 degrees
- moved C1 17.8 mm to (213.2, 64.0), turned to 90 degrees
- moved D7 16.1 mm to (220.5, 65.8), turned to 90 degrees
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Routing:
- net GND: track 0.00 -> 319.9 mm, vias 0 -> 1
- net FLEXIBLE_IO_10: track 115.2 -> 50.4 mm
- net FLEXIBLE_IO_11: track 99.9 -> 43.6 mm
- net CONTROL_RELAY_GROUP_ONE: track 47.0 -> 101.6 mm
- net IN_BOILER_PROBE: track 81.1 -> 134.9 mm
- net +3.3V: track 211.7 -> 165.9 mm, vias 2 -> 1
- net FLEXIBLE_IO_12: track 56.0 -> 13.7 mm
- net CONTROL_RELAY_TEA: track 41.5 -> 79.8 mm, vias 0 -> 1
- net OUT_BOILER_PROBE_VOLTAGE: track 18.2 -> 55.9 mm
- net SOL_L: track 70.9 -> 38.2 mm, vias 0 -> 1
- net FLEXIBLE_IO_03: track 38.6 -> 71.2 mm
- net AC_SOLENOID_PHASE: track 103.8 -> 71.3 mm
- net FLEXIBLE_IO_05: track 33.6 -> 65.5 mm, vias 0 -> 1
- net FLEXIBLE_IO_06: track 37.6 -> 66.2 mm
- net FLEXIBLE_IO_09: track 39.4 -> 12.0 mm
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- removed copper zone on B.Cu, net GND
Other:
- board size 113 x 129 mm -> 87.5 x 129 mm
- board text removed: "+5V"
- board text removed: "1 RAW"
- board text removed: "1 SOL-L"
- board text removed: "2 +5V"
- board text removed: "2 AC-L"
- board text removed: "C1 1n G1"
- board text removed: "C2 1n G2"
- board text removed: "D6 ESD G1"
- board text removed: "D7 ESD G2"
- board text removed: "GND"
- board text removed: "H1 M3"
- board text removed: "H2 M3"
- board text removed: "H3 M3"
- board text removed: "H4 M3"
- board text removed: "J1 5V IN"
- board text removed: "J11 SOL FUSE"
- board text removed: "J12 5V FUSE"
- board text removed: "J13 I2C"
- board text removed: "R5 10k BP"
- board text removed: "R7 10k BP"
- board text removed: "R8 10k FM2"
- board text removed: "R9 10k FM1"

Commit message: BrewPilot Volume 2 - The Pilot returns as Compact
Parts:
- moved J11 30.3 mm to (170.5, 108.0), turned to 0 degrees
- moved H4 20.5 mm to (225.0, 140.0)
- moved K5 19.9 mm to (190.0, 128.8)
- moved K4 19.8 mm to (199.1, 128.9)
- moved K3 19.7 mm to (208.0, 128.9)
- moved K1 19.6 mm to (218.1, 129.1)
- moved K2 19.5 mm to (227.1, 129.1)
- moved H3 19.0 mm to (151.5, 140.5)
- moved J6 18.4 mm to (162.8, 140.6)
- moved J7 18.4 mm to (186.9, 140.6)
- moved J8 18.4 mm to (204.2, 140.5)
- moved J9 18.4 mm to (213.7, 140.5)
- moved Q5 16.7 mm to (187.3, 104.0)
- moved Q4 16.0 mm to (196.3, 104.1)
- moved Q1 15.9 mm to (215.3, 104.1)
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Routing:
- net +5V: track 218.8 -> 150.8 mm
- net SOL_L: track 38.2 -> 86.4 mm, vias 1 -> 0
- net CONTROL_RELAY_GROUP_ONE: track 101.6 -> 53.7 mm, vias 1 -> 3
- net IN_BOILER_PROBE: track 134.9 -> 107.3 mm, vias 0 -> 1
- net OUT_BOILER_PROBE_VOLTAGE: track 55.9 -> 79.7 mm
- net CONTROL_RELAY_TEA: track 79.8 -> 59.2 mm, vias 1 -> 0
- net CONTROL_RELAY_PUMP: track 75.3 -> 56.6 mm, vias 1 -> 0
- net FLEXIBLE_IO_03: track 71.2 -> 55.4 mm
- net AC_SOLENOID_PHASE: track 71.3 -> 82.7 mm, vias 0 -> 1
- net FLEXIBLE_IO_08: track 71.8 -> 83.1 mm, vias 1 -> 2
- net FLEXIBLE_IO_05: track 65.5 -> 54.6 mm, vias 1 -> 0
- net +3.3V: track 165.9 -> 176.7 mm
- net AC_SOLENOID_GROUP_TWO: track 50.8 -> 40.5 mm, vias 1 -> 0
- net CONTROL_RELAY_BOILER_FILL: track 78.6 -> 69.8 mm
- net IN_FLOWMETER_GROUP_TWO: track 100.4 -> 93.0 mm
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Other:
- board size 87.5 x 129 mm -> 87.5 x 111 mm
- board text added: "BLR FILL"
- board text added: "GRP1"
- board text added: "GRP2"
- board text added: "PUMP"
- board text added: "R1 4k7"
- board text added: "R10 1K"
- board text added: "R11 1K"
- board text added: "R12 1K"
- board text added: "R13 1K"
- board text added: "R14 1K"
- board text added: "R2 4k7"
- board text added: "R3 4k7"
- board text added: "R4 4k7"
- board text added: "R6 4k7"
- board text added: "TEA"
- board text removed: "D1 PUMP"
- board text removed: "D2 FILL"
- board text removed: "D3 G1"
- board text removed: "D4 G2"
- board text removed: "D5 TEA"
- board text removed: "K1 PUMP"
- board text removed: "K2 FILL"
- board text removed: "K3 G1"
- board text removed: "K4 G2"
- board text removed: "K5 TEA"
- board text removed: "Q1 PUMP"
- board text removed: "Q2 FILL"
- board text removed: "Q3 G1"
- board text removed: "Q4 G2"
- board text removed: "Q5 TEA"
- board text removed: "R1 4k7 FILL"
- board text removed: "R10 1k PUMP"
- board text removed: "R11 1k FILL"
- board text removed: "R12 1k G1"
- board text removed: "R13 1k G2"
- board text removed: "R14 1k TEA"
- board text removed: "R2 4k7 G1"
- board text removed: "R3 4k7 G2"
- board text removed: "R4 4k7 TEA"
- board text removed: "R6 4k7 PUMP"

Commit message: Save current BrewPilot PCB design before schematic alignment
Amp-Thread-ID: https://ampcode.com/threads/T-01a0debc-596d-7434-9824-16fe8385066c
Co-authored-by: Amp <amp@ampcode.com>
Parts:
- J11: footprint new_local:696108003002 -> new_local:BLX-A_5x20mm
- J12: footprint Fuse:Fuseholder_Cylinder-5x20mm_Schurter_0031_8201_Horizontal_Open -> new_local:BLX-A_5x20mm
- Q1, Q2, Q3, Q4, Q5: footprint Package_TO_SOT_THT:TO-92_Inline -> Package_TO_SOT_THT:TO-92_Inline_Wide
- moved J11 16.5 mm to (171.0, 124.5)
- moved K2 2.00 mm to (225.1, 129.1)
- moved Q1 1.27 mm to (214.1, 104.1)
- moved Q2 1.27 mm to (223.1, 104.1)
- moved Q3 1.27 mm to (204.1, 104.1)
- moved Q4 1.27 mm to (195.1, 104.1)
- moved Q5 1.27 mm to (186.1, 104.0)
- moved K5 0.50 mm to (190.0, 129.3)
Routing:
- net FLEXIBLE_IO_04: track 55.7 -> 120.0 mm
- net FLEXIBLE_IO_03: track 55.4 -> 110.2 mm
- net AC_SOLENOID_PHASE: track 82.7 -> 48.2 mm, vias 1 -> 0
- net CONTROL_RELAY_GROUP_TWO: track 66.5 -> 99.5 mm, vias 0 -> 2
- net FLEXIBLE_IO_07: track 64.9 -> 95.3 mm
- net GND: track 320.9 -> 349.9 mm
- net OUT_BOILER_PROBE_VOLTAGE: track 79.7 -> 57.3 mm, vias 0 -> 1
- net +5V: track 150.8 -> 171.0 mm
- net IN_FLOWMETER_GROUP_TWO: track 93.0 -> 106.9 mm
- net CONTROL_RELAY_PUMP: track 56.6 -> 70.3 mm
- net SOL_L: track 86.4 -> 72.7 mm
- net FLEXIBLE_IO_05: track 54.6 -> 65.4 mm
- net CONTROL_RELAY_TEA: track 59.2 -> 67.0 mm, vias 0 -> 1
- net FLEXIBLE_IO_10: track 50.4 -> 58.1 mm
- net IN_FLOWMETER_GROUP_ONE: track 54.2 -> 61.2 mm, vias 1 -> 0
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- added copper zone on B.Cu, net GND
- added copper zone on F.Cu, net GND
Other:
- board text added: "USB -->"
- board text added: "brewpilot v0.1"
- board text added: "by ben & niklas"
- board text added: "reingeguckt"

Commit message: ai driven improvements
Other:
- board text added: "brewpilot v0.2"
- board text removed: "brewpilot v0.1"

Commit message: migrated ssrs to their own assembly
Parts:
- moved K2 10.9 mm to (214.2, 129.0)
- moved R1 10.1 mm to (214.0, 99.9)
- moved D2 10.0 mm to (214.3, 88.8)
- moved Q2 10.0 mm to (213.1, 104.1)
- moved R11 9.90 mm to (217.2, 99.9)
- moved R10 8.10 mm to (226.2, 99.9)
- moved Q1 8.00 mm to (222.1, 104.1)
- moved D1 8.00 mm to (223.3, 88.8)
- moved R6 7.90 mm to (223.0, 99.9)
- moved K1 5.10 mm to (223.2, 129.0)
- moved K4 2.90 mm to (196.2, 129.0)
- moved K5 2.81 mm to (187.2, 129.0)
- moved K3 2.80 mm to (205.2, 129.0)
- moved R13 0.39 mm to (199.2, 99.9)
- moved D5 0.30 mm to (187.3, 88.8)
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Routing:
- net GND: track 349.9 -> 285.8 mm
- net AC_SOLENOID_PHASE: track 48.2 -> 35.2 mm
- net AC_SOLENOID_BOILER_FILL: track 38.0 -> 25.9 mm
- net AC_SOLENOID_GROUP_TWO: track 33.6 -> 44.5 mm
- net AC_SOLENOID_NEUTRAL: track 61.1 -> 68.5 mm
- net CONTROL_RELAY_PUMP: track 70.3 -> 77.6 mm, vias 0 -> 1
- net AC_PUMP_POWER_OUT: track 39.3 -> 45.8 mm
- net +5V: track 171.0 -> 174.9 mm
- net AC_SOLENOID_TEA: track 35.6 -> 33.0 mm
- net SSR_PUMP_SINK: track 24.1 -> 21.7 mm
- net AC_PUMP_NEUTRAL: track 32.5 -> 34.7 mm
- net AC_PUMP_PHASE: track 11.7 -> 13.9 mm
- net CONTROL_RELAY_GROUP_TWO: track 99.5 -> 101.5 mm
- net CONTROL_RELAY_GROUP_ONE: track 55.1 -> 57.0 mm
- net SSR_TEA_SINK: track 23.4 -> 21.7 mm
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
Commit message: Checkpoint current PCB revision and machine-specific firmware builds
Preserve the existing workspace before firmware safety fixes.

Amp-Thread-ID: https://ampcode.com/threads/T-01a12a1e-8ea4-702d-96da-3a9264193d9b
Co-authored-by: Amp <amp@ampcode.com>
Parts:
- added R17: 4.7k, Resistor_THT:R_Axial_DIN0207_L6.3mm_D2.5mm_P7.62mm_Horizontal, F.Cu at (221.0, 99.9)
- added R18: 4.7k, Resistor_THT:R_Axial_DIN0207_L6.3mm_D2.5mm_P7.62mm_Horizontal, F.Cu at (210.2, 99.9)
- added R19: 4.7k, Resistor_THT:R_Axial_DIN0207_L6.3mm_D2.5mm_P7.62mm_Horizontal, F.Cu at (199.4, 99.9)
- added R20: 4.7k, Resistor_THT:R_Axial_DIN0207_L6.3mm_D2.5mm_P7.62mm_Horizontal, F.Cu at (188.6, 99.9)
- added R21: 4.7k, Resistor_THT:R_Axial_DIN0207_L6.3mm_D2.5mm_P7.62mm_Horizontal, F.Cu at (177.8, 99.9)
- added R22: 10k, Resistor_THT:R_Axial_DIN0207_L6.3mm_D2.5mm_P7.62mm_Horizontal, F.Cu at (175.2, 57.0)
- added R23: 10k, Resistor_THT:R_Axial_DIN0207_L6.3mm_D2.5mm_P7.62mm_Horizontal, F.Cu at (180.0, 57.0)
- added R24: 10k, Resistor_THT:R_Axial_DIN0207_L6.3mm_D2.5mm_P7.62mm_Horizontal, F.Cu at (160.8, 57.0)
- added R25: 10k, Resistor_THT:R_Axial_DIN0207_L6.3mm_D2.5mm_P7.62mm_Horizontal, F.Cu at (189.6, 57.0)
- added R26: 10k, Resistor_THT:R_Axial_DIN0207_L6.3mm_D2.5mm_P7.62mm_Horizontal, F.Cu at (194.4, 57.0)
- added R27: 10k, Resistor_THT:R_Axial_DIN0207_L6.3mm_D2.5mm_P7.62mm_Horizontal, F.Cu at (199.2, 57.0)
- J13: footprint Connector_RJ:RJ45_Amphenol_54602-x08_Horizontal -> new_local:RJ45_Amphenol_54602-x08_BoardEdge
- moved R8 35.2 mm to (184.8, 64.6), turned to 90 degrees
- moved J11 8.20 mm to (162.8, 124.5)
- moved K5 7.20 mm to (180.0, 129.0)
- moved Q5 7.20 mm to (178.9, 104.1)
- moved R4 5.60 mm to (181.4, 99.9)
- moved R9 5.53 mm to (204.0, 64.6), turned to 90 degrees
- moved Q4 5.40 mm to (189.7, 104.1)
- moved K4 5.40 mm to (190.8, 129.0)
- moved R14 5.20 mm to (185.0, 99.9)
- moved D5 4.80 mm to (182.5, 88.8)
- moved R16 4.64 mm to (165.6, 57.0)
- moved R15 4.51 mm to (170.4, 57.0)
- moved R3 3.80 mm to (192.2, 99.9)
- moved K3 3.60 mm to (201.6, 129.0)
- moved Q3 3.60 mm to (200.5, 104.1)
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Connections:
- J13 pad 1: FLEXIBLE_IO_10 -> I2C_SDA
- J13 pad 2: FLEXIBLE_IO_11 -> I2C_SCL
- R15 pad 2: FLEXIBLE_IO_10 -> I2C_SDA
- R16 pad 2: FLEXIBLE_IO_11 -> I2C_SCL
- U1 pad 12: FLEXIBLE_IO_03 -> FLEXIBLE_IO_11
- U1 pad 15: FLEXIBLE_IO_01 -> FLEXIBLE_IO_10
- U1 pad 3: unconnected-(U1-GPI36-Pad3) -> FLEXIBLE_IO_01
- U1 pad 33: FLEXIBLE_IO_10 -> I2C_SDA
- U1 pad 36: FLEXIBLE_IO_11 -> I2C_SCL
- U1 pad 4: unconnected-(U1-GPI39-Pad4) -> FLEXIBLE_IO_03
Routing:
- net GND: track 285.8 -> 75.8 mm, vias 0 -> 12
- net FLEXIBLE_IO_11: track 43.6 -> 110.5 mm, vias 0 -> 1
- net CONTROL_RELAY_TEA: track 67.2 -> 132.2 mm
- net FLEXIBLE_IO_03: track 110.2 -> 58.2 mm
- net FLEXIBLE_IO_08: track 86.0 -> 123.0 mm, vias 1 -> 2
- net I2C_SDA: track 0.00 -> 35.1 mm
- net I2C_SCL: track 0.00 -> 27.7 mm
- net FLEXIBLE_IO_07: track 95.3 -> 69.1 mm, vias 1 -> 0
- net CONTROL_RELAY_GROUP_ONE: track 57.0 -> 83.2 mm, vias 0 -> 1
- net FLEXIBLE_IO_02: track 59.5 -> 84.9 mm, vias 1 -> 0
- net FLEXIBLE_IO_05: track 65.4 -> 87.5 mm, vias 0 -> 2
- net IN_BOILER_PROBE: track 108.9 -> 126.9 mm, vias 0 -> 2
- net +3.3V: track 170.9 -> 153.0 mm, vias 0 -> 1
- net FLEXIBLE_IO_10: track 58.1 -> 76.0 mm, vias 0 -> 2
- net FLEXIBLE_IO_12: track 13.7 -> 30.3 mm, vias 0 -> 1
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Other:
- board text added: "1 SDA"
- board text added: "2 SCL"
- board text added: "R15 4k7 SDA"
- board text added: "R16 4k7 SCL"
- board text added: "R17 4k7"
- board text added: "R18 4k7"
- board text added: "R19 4k7"
- board text added: "R20 4k7"
- board text added: "R21 4k7"
- board text added: "R22 10k IO1"
- board text added: "R23 10k IO3"
- board text added: "R24 10k IO12"
- board text added: "R25 10k IO6"
- board text added: "R26 10k IO5"
- board text added: "R27 10k IO4"
- board text added: "R8 10k FLOW2"
- board text added: "R9 10k FLOW1"
- board text added: "brewpilot v0.3"
- board text removed: "1 IO10"
- board text removed: "2 IO11"
- board text removed: "R15 4k7 IO10"
- board text removed: "R16 4k7 IO11"
- board text removed: "brewpilot v0.2"
